Commit message: visualization without tracking

File: rrr_challenge/include/rrr_challenge/urdf/rrr.urdf (robot description, URDF)
Before this commit: robot rrr_robot, 5 links, 4 joints
Links:
- removed link base_link
- added link end_effector_tip; visual sphere radius=0.02
- link base_joint_link: geometry collision mesh filename=package://rrr_challenge/urdf/mesh/base_joint.stl scale=1 1 1; visual mesh filename=package://rrr_challenge/urdf/mesh/base_joint.stl scale=1 1 1
- link link1: geometry collision mesh filename=package://rrr_challenge/urdf/mesh/first_arm.stl scale=1 1 1; visual mesh filename=package://rrr_challenge/urdf/mesh/first_arm.stl scale=1 1 1
- link link2: geometry collision mesh filename=package://rrr_challenge/urdf/mesh/second_arm.stl scale=1 1 1; visual mesh filename=package://rrr_challenge/urdf/mesh/second_arm.stl scale=1 1 1
- link link3: geometry collision mesh filename=package://rrr_challenge/urdf/mesh/third_arm.stl scale=1 1 1; visual mesh filename=package://rrr_challenge/urdf/mesh/third_arm.stl scale=1 1 1
Joints:
- removed joint base_to_base_joint
- added joint end_effector_fixed_joint: type fixed, parent link3, child end_effector_tip, origin xyz=0 0.27 1 rpy=0 0 0
- joint joint1: axis 0 0 1 -> 0 1 0; origin xyz=0 0 0.1 rpy=0 0 0 -> xyz=0 -0.175 0 rpy=0 0 0
- joint joint2: origin xyz=0.2 0 0 rpy=0 0 0 -> xyz=0 0.3 1 rpy=0 0 0
- joint joint3: origin xyz=0.2 0 0 rpy=0 0 0 -> xyz=0 -0.3 1 rpy=0 0 0

Commit message: solve the reference system issue

File: rrr_challenge/include/rrr_challenge/urdf/rrr.urdf (robot description, URDF)
Before this commit: robot rrr_robot, 5 links, 4 joints
Links:
- added link world
Joints:
- added joint world_to_base: type fixed, parent world, child base_joint_link, origin xyz=0 0 0 rpy=0 1.5708 3.141592

Commit message: working

File: rrr_challenge/include/rrr_challenge/urdf/rrr.urdf (robot description, URDF)
Before this commit: robot rrr_robot, 6 links, 5 joints
Joints:
- joint world_to_base: origin xyz=0 0 0 rpy=0 1.5708 3.141592 -> xyz=0 0 0 rpy=0 -1.5708 3.141592

Commit message: added disk

File: rrr_challenge/include/rrr_challenge/urdf/rrr.urdf (robot description, URDF)
Before this commit: robot rrr_robot, 6 links, 5 joints
Links:
- added link constraint_disk, mass 0.0001; visual cylinder length=0.01 radius=0.25
Joints:
- added joint constraint_disk_joint: type fixed, parent base_joint_link, child constraint_disk, origin xyz=0.5 0 1 rpy=0 0 0
